Commit message: add border

File: src/xarm7_mov_test/urdf/xarm7_with_gripper.xacro (robot description, xacro)
@@ -7,5 +7,5 @@
   <xacro:include filename="$(find xarm_description)/urdf/xarm7_robot_macro.xacro" />
   <xacro:xarm7_robot prefix="$(arg prefix)" namespace="$(arg ros_namespace)" limited="$(arg limited)" effort_control="$(arg effort_control)"
-  attach_to="base_link" xyz="0 0 0.15" rpy="0 0 1.57"/>
+  attach_to="base_link" xyz="0.7 0.5 0.15" rpy="0 0 -0.52"/>
 <xacro:include filename="$(find xarm_gripper)/urdf/xarm_gripper_model.xacro" />
 <xacro:load_gripper prefix="$(arg prefix)" effort_control="$(arg effort_control)"
@@ -22,4 +22,32 @@
     <material name="blue"/>
   </visual>
+  <visual>
+    <origin rpy="0 0 0" xyz="0 0.75 0.3"/>
+    <geometry>
+      <box size="2 0.05 0.3"/>
+    </geometry>
+    <material name="blue"/>
+  </visual>
+ <visual>
+    <origin rpy="0 0 0" xyz="0 -0.75 0.3"/>
+    <geometry>
+      <box size="2 0.05 0.3"/>
+    </geometry>
+    <material name="blue"/>
+  </visual>
+   <visual>
+    <origin rpy="0 0 0" xyz="1 0 0.3"/>
+    <geometry>
+      <box size="0.05 1.5 0.3"/>
+    </geometry>
+    <material name="blue"/>
+  </visual>
+  <visual>
+    <origin rpy="0 0 0" xyz="-1 0 0.3"/>
+    <geometry>
+      <box size="0.05 1.5 0.3"/>
+    </geometry>
+    <material name="blue"/>
+  </visual>
 </link>
 <link name="tool_0">
