Commit message: ur5 with kinova
ur5 with kinova

File: src/ur_description_robots/urdf/ur5_with_base_prev.xacro (robot description, xacro)
@@ -23,37 +23,9 @@
       <material name="blue"/>
     </visual>
-  <visual>
-    <origin rpy="0 0 0" xyz="0 0.75 0.3"/>
-    <geometry>
-      <box size="2 0.05 0.3"/>
-    </geometry>
-    <material name="blue"/>
-  </visual>
- <visual>
-    <origin rpy="0 0 0" xyz="0 -0.75 0.3"/>
-    <geometry>
-      <box size="2 0.05 0.3"/>
-    </geometry>
-    <material name="blue"/>
-  </visual>
-   <visual>
-    <origin rpy="0 0 0" xyz="1 0 0.3"/>
-    <geometry>
-      <box size="0.05 1.5 0.3"/>
-    </geometry>
-    <material name="blue"/>
-  </visual>
-  <visual>
-    <origin rpy="0 0 0" xyz="-1 0 0.3"/>
-    <geometry>
-      <box size="0.05 1.5 0.3"/>
-    </geometry>
-    <material name="blue"/>
-  </visual>
   </link>
   <joint name="world_joint_table" type="fixed">
     <parent link="base_table"/>
     <child link="base_link"/>
-    <origin xyz="0.7 -0.5 0.15" rpy="0.0 0.0 0.9"/>
+    <origin xyz="0.0 0.0 0.15" rpy="0.0 0.0 0.0"/>
   </joint>
 </robot>
